File: TranceiverV1/TranceiverV1.kicad_pcb (KiCad board)
At the start: 2 copper layers, 94.6 x 45.6 mm, 19 parts, among them J1 Conn_01x03_Socket, J3 Battery, SW1 SW_Push_Open, U1 NRF24L01_, U3 102010388, U4 LD1086DTTR

Commit message: changed switch
Parts:
- removed SW1: SW_Push_Open, Button_Switch_THT:SW_PUSH_1P1T_6x3.5mm_H5.0_APEM_MJTP1250
- added S3: ATE1D-2M3-10-Z, ATE1D-2M3-10-Z:SW_ATE1D-2M3-10-Z, F.Cu at (126.2, 129.5)
Connections:
- U1 pad 1: GND -> (no net)
- U1 pad 2: /VCC -> (no net)
- U1 pad 3: /CE -> (no net)
- U1 pad 4: /CSN -> (no net)
- U1 pad 5: /SCK -> (no net)
- U1 pad 6: /MOSI -> (no net)
- U1 pad 7: /MISO -> (no net)
- U1 pad 8: IRQ -> (no net)
Routing:
- net Net-(J3-Pin_1): track 8.46 -> 16.6 mm
- net /Regulator_In: track 30.5 -> 27.5 mm
