File: ReceiverModule/ReceiverModule.kicad_pcb (KiCad board)
At the start: 2 copper layers, 94.6 x 45.6 mm, 23 parts, among them J1 Conn_01x03_Socket, J3 Battery, U1 NRF24L01_, U3 102010388, U4 LD1086DTTR

Commit message: added net id and name
Other:
- board text added: "ag821 Alisha Gupta"
Changed lines of the file:
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@@
 		(layer "Edge.Cuts")
+	)
+	(gr_text "ag821 Alisha Gupta"
+		(at 177.1 142.3 0)
+		(layer "F.Cu")
+		(effects
+			(font
+				(size 1.5 1.5)
+				(thickness 0.3)
+				(bold yes)
+			)
+			(justify left bottom)
+		)
 	)
 	(segment
